File: newMain.brd (EAGLE design)
At the start: 82.2 x 74.9 mm, 15 parts, among them M1 SERVO, M2 SERVO

Commit message: pcb
Parts:
- removed J1: (no value), SparkFun-Connectors:1X04
- removed J5, J6: (no value), SparkFun-Retired:1X02_2.54_SCREWTERM
- added SV1: (no value), con-lstb:MA10-1W
- moved R2 41.9 mm to (77.5, 39.4), turned to 270 degrees
- moved MOTOR 27.4 mm to (59.7, 36.8), turned to 90 degrees
- moved MAIN_MCU 26.9 mm to (50.8, 20.3)
- moved R1 26.5 mm to (30.5, 38.1), turned to 90 degrees
- moved R3 26.1 mm to (68.6, 39.4), turned to 270 degrees
- moved U$1 25.7 mm to (95.2, 20.3), turned to 270 degrees
- moved J2 24.4 mm to (40.6, 39.4)
- moved J3 21.9 mm to (47.0, 41.9)
- moved MOTOR_PWR 15.5 mm to (19.1, 6.35), turned to 180 degrees
- moved M1 14.2 mm to (21.6, 41.9)
- moved MCU_PWR 8.89 mm to (30.5, 6.35), turned to 180 degrees
- moved M2 8.03 mm to (21.6, 27.9)
Connections:
- removed net DATA_RF: J1.3
- new net B0: MAIN_MCU.J2.12, SV1.2
- new net B1: MAIN_MCU.J2.11, SV1.3
- new net B2: MAIN_MCU.J2.10, SV1.4
- new net B3: MAIN_MCU.J2.9, SV1.5
- new net B4: MAIN_MCU.J2.8, SV1.6
- new net B5: MAIN_MCU.J2.7, SV1.7
- net GND: now also SV1.10; no longer J1.4
- net RX_BLE: now also MAIN_MCU.J1.11
- net TX_BLE: now also MAIN_MCU.J1.10
- net VCC_2: now also SV1.1; no longer J1.1
Routing:
- net VCC_2: track 292.7 -> 185.1 mm
- net N$5: track 62.6 -> 10.2 mm
- net RX_BLE: track 0.00 -> 47.1 mm
- net GND: track 262.0 -> 233.2 mm
- net TX_MAIN: track 24.0 -> 0.00 mm
- net DATA_RF: track 15.0 -> 0.00 mm
- net B4: track 0.00 -> 12.1 mm
- net B3: track 0.00 -> 10.8 mm
- net B2: track 0.00 -> 10.8 mm
- net B5: track 0.00 -> 10.8 mm
- net B1: track 0.00 -> 10.8 mm
- net B0: track 0.00 -> 10.8 mm
- net RX_MAIN: track 10.2 -> 0.00 mm
- net OPT: track 11.0 -> 21.1 mm
- net SEV_1: track 48.2 -> 39.7 mm
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- added copper zone on layer 16, net N$1
- removed copper zone on layer 16, net N$13
Other:
- board size 82.2 x 74.9 mm -> 74.6 x 47 mm
- board text removed: "+"
- board text removed: "+ - TX RX"
- board text removed: "5V"
- board text removed: "7V"
- board text removed: "EN"
- board text removed: "MAGNET"
- board text removed: "MAIN FOR FB"
- board text removed: "RF315"
